Commit message: Figured out bug, generated code for cartpole, need kinematics and wrapper

File: models/cartpole/cartpole.urdf (robot description, URDF)
Before this commit: robot physics, 3 links, 2 joints
Links:
- added link pole_tip
Joints:
- added joint pole_to_cart: type fixed, parent pole, child pole_tip, origin xyz=0 0 1
- joint cart_to_pole: limit (none) -> effort=1000.0 velocity=5; type continuous -> revolute

Commit message: Updated cartpole inertial and visual properties

File: models/cartpole/cartpole.urdf (robot description, URDF)
Before this commit: robot physics, 4 links, 3 joints
Links:
- link pole: mass 10 -> 1
- link pole_tip: geometry visual sphere radius=0.1
