Commit message: Small bug fixes, demoed that most pinocchio funcs aren't reliable with non-unit quats

File: models/nadia/nadiaV17.fullRobot.simpleKnees.cycloidArms_mj.urdf (robot description, URDF)
Before this commit: robot nadia, 45 links, 44 joints
Links:
- link LEFT_ANKLE_LINK: geometry visual mesh filename=package://nadia_V16_description/meshes/ankle.obj
- link LEFT_ELBOW_PITCH_LINK: geometry visual mesh filename=package://nadia_V17_description/meshes/cycloidal_arm/LEFT_E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
- link LEFT_FOOT_LINK: geometry visual mesh filename=package://nadia_V16_description/meshes/foot.obj
- link LEFT_HIP_ROLL_LINK: geometry visual mesh filename=package://nadia_V16_description/meshes/left_hip_roll.obj
- link LEFT_HIP_YAW_LINK: geometry visual mesh filename=package://nadia_V16_description/meshes/left_hip_yaw.obj
- link LEFT_SHIN_LINK: geometry visual mesh filename=package://nadia_V16_description/meshes/left_shin.obj
- link LEFT_SHOULDER_PITCH_LINK: geometry visual mesh filename=package://nadia_V17_description/meshes/cycloidal_arm/LEFT_S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
- link LEFT_SHOULDER_ROLL_LINK: geometry visual mesh filename=package://nadia_V17_description/meshes/cycloidal_arm/LEFT_S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
- link LEFT_SHOULDER_YAW_LINK: geometry visual mesh filename=package://nadia_V17_description/meshes/cycloidal_arm/LEFT_S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
- link LEFT_THIGH_LINK: geometry visual mesh filename=package://nadia_V16_description/meshes/left_thigh.obj
- link PELVIS_LINK: geometry visual mesh filename=package://nadia_V16_description/meshes/pelvis.obj
- link RIGHT_ANKLE_LINK: geometry visual mesh filename=package://nadia_V16_description/meshes/ankle.obj
- link RIGHT_ELBOW_PITCH_LINK: geometry visual mesh filename=package://nadia_V17_description/meshes/cycloidal_arm/RIGHT_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
- link RIGHT_FOOT_LINK: geometry visual mesh filename=package://nadia_V16_description/meshes/foot.obj
- link RIGHT_HIP_ROLL_LINK: geometry visual mesh filename=package://nadia_V16_description/meshes/right_hip_roll.obj
- link RIGHT_HIP_YAW_LINK: geometry visual mesh filename=package://nadia_V16_description/meshes/right_hip_yaw.obj
- link RIGHT_SHIN_LINK: geometry visual mesh filename=package://nadia_V16_description/meshes/right_shin.obj
- link RIGHT_SHOULDER_PITCH_LINK: geometry visual mesh filename=package://nadia_V17_description/meshes/cycloidal_arm/RIGHT_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
- link RIGHT_SHOULDER_ROLL_LINK: geometry visual mesh filename=package://nadia_V17_description/meshes/cycloidal_arm/RIGHT_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
- link RIGHT_SHOULDER_YAW_LINK: geometry visual mesh filename=package://nadia_V17_description/meshes/cycloidal_arm/RIGHT_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
- link RIGHT_THIGH_LINK: geometry visual mesh filename=package://nadia_V16_description/meshes/right_thigh.obj
- link SPINE_ROLL_LINK: geometry visual mesh filename=package://nadia_V16_description/meshes/spine_roll.obj
- link SPINE_YAW_LINK: geometry visual mesh filename=package://nadia_V16_description/meshes/spine_yaw.obj
- link TORSO_LINK: geometry visual mesh filename=package://nadia_V16_description/meshes/torso_cycloidmounts.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
