Commit message: Changed arms so they aren't straight down, dynamics need to be regenerated

File: models/nadia/nadiaV17.fullRobot.simpleKnees.fixedArms_mj.urdf (robot description, URDF)
Before this commit: robot nadia, 45 links, 44 joints
Joints:
- joint LEFT_ELBOW_Y: origin xyz=0.015 0.0 -0.4 rpy=0.0 0.0 0.0 -> xyz=0.015 0.0 -0.4 rpy=0.0 -1.396 0.0
- joint LEFT_SHOULDER_X: origin xyz=0.0 0.15676000 -0.01300000 rpy=-0.785398163 0.0 0.0 -> xyz=0.0 0.15676000 -0.01300000 rpy=-0.531398163 0.0 0.0
- joint LEFT_SHOULDER_Y: origin xyz=0.001 0.185 0.173 rpy=0.785398163 0.0 -0.785398163 -> xyz=0.001 0.185 0.173 rpy=0.785398163 0.387 -0.785398163
- joint RIGHT_ELBOW_Y: origin xyz=0.015 0.0 -0.4 rpy=0.0 0.0 0.0 -> xyz=0.015 0.0 -0.4 rpy=0.0 -1.396 0.0
- joint RIGHT_SHOULDER_X: origin xyz=0.0 -0.15676000 -0.01300000 rpy=0.785398163 0.0 0.0 -> xyz=0.0 -0.15676000 -0.01300000 rpy=0.531398163 0.0 0.0
- joint RIGHT_SHOULDER_Y: origin xyz=0.001 -0.185 0.173 rpy=-0.785398163 0.0 0.785398163 -> xyz=0.001 -0.185 0.173 rpy=-0.785398163 0.387 0.785398163
