Commit message: Added double cartpole, changed cartpole to slide along y, rotate around x

File: models/double_cartpole/double_cartpole.urdf (robot description, URDF)
Before this commit: robot physics, 4 links, 3 joints
Links:
- removed link pole
- added link pole1, mass 1; collision box size=0.05 0.05 1.0; visual cylinder length=1 radius=0.04
- added link pole2, mass 1; collision box size=0.05 0.05 1.0; visual cylinder length=1 radius=0.04
Joints:
- removed joint pole_to_cart
- added joint pole2: type revolute, parent pole1, child pole2, origin xyz=0.0 0.0 1.0, axis 1 0 0, limit effort=1000.0 velocity=5
- added joint tip_joint: type fixed, parent pole2, child pole_tip, origin xyz=0 0 1
- joint cart_to_pole: child pole -> pole1
