Commit message: Update pineapple

File: models/pineapple/pineapple_8dof.urdf (robot description, URDF)
Before this commit: robot pineapple_8dof, 12 links, 11 joints
Links:
- removed link L_hip_fix
- removed link R_hip_fix
- removed link battery
- added link depth_cam, mass 0.30000000; visual mesh filename=package://v1/meshes/depth_cam.STL
- link L_calf: mass 0.555 -> 0.50000000; geometry collision mesh filename=package://v1/meshes/L_calf_collision.STL; visual mesh filename=package://v1/meshes/L_calf.STL
- link L_hip: mass 0.573 -> 0.57300000; geometry visual mesh filename=package://v1/meshes/L_hip.STL
- link L_thigh: mass 0.9105 -> 0.75000000; geometry collision mesh filename=package://v1/meshes/L_thigh_collision.STL; visual mesh filename=package://v1/meshes/L_thigh.STL
- link L_wheel: mass 0.2805 -> 0.30500000; geometry collision cylinder length=0.026 radius=0.075; visual mesh filename=package://v1/meshes/L_wheel.STL
- link R_calf: mass 0.555 -> 0.50000000; geometry collision mesh filename=package://v1/meshes/R_calf_collision.STL; visual mesh filename=package://v1/meshes/R_calf.STL
- link R_hip: mass 0.573 -> 0.57300000; geometry visual mesh filename=package://v1/meshes/R_hip.STL
- link R_thigh: mass 0.9105 -> 0.75000000; geometry collision mesh filename=package://v1/meshes/R_thigh_collision.STL; visual mesh filename=package://v1/meshes/R_thigh.STL
- link R_wheel: mass 0.2805 -> 0.30500000; geometry collision cylinder length=0.026 radius=0.075; visual mesh filename=package://v1/meshes/R_wheel.STL
- link base_link: mass 0.62 -> 2.85000000; geometry collision mesh filename=package://v1/meshes/base_collision.STL; visual mesh filename=package://v1/meshes/base_link.STL
Joints:
- removed joint L_base2hip
- removed joint L_calf2wheel
- removed joint L_hip2thigh
- removed joint L_hip_fix
- removed joint L_thigh2calf
- removed joint R_base2hip
- removed joint R_calf2wheel
- removed joint R_hip2thigh
- removed joint R_hip_fix
- removed joint R_thigh2calf
- removed joint battery_fix
- added joint L_calf_joint: type revolute, parent L_thigh, child L_calf, origin xyz=0 0.0388671106492234 -0.190000930017623 rpy=0 0 0, axis 0 1 0, limit lower=-3.1416 upper=0.0 effort=33.5 velocity=21.0
- added joint L_hip_joint: type revolute, parent base_link, child L_hip, origin xyz=0 0.061249999999998 0.0610009280869146 rpy=0 0 0, axis 1 0 0, limit lower=-0.52358 upper=0.17444 effort=23.7 velocity=30.0
- added joint L_thigh_joint: type revolute, parent L_hip, child L_thigh, origin xyz=0 0.01 0 rpy=0 0 0, axis 0 1 0, limit lower=0.0 upper=1.571 effort=23.7 velocity=30.0
- added joint L_wheel_joint: type revolute, parent L_calf, child L_wheel, origin xyz=0 0.0421817545313912 -0.190000000000001 rpy=0 0 0, axis 0 1 0, limit effort=3.69 velocity=60.0
- added joint R_calf_joint: type revolute, parent R_thigh, child R_calf, origin xyz=0 -0.0388671106492234 -0.190000930017624 rpy=0 0 0, axis 0 1 0, limit lower=-3.1416 upper=0.0 effort=33.5 velocity=21.0
- added joint R_hip_joint: type revolute, parent base_link, child R_hip, origin xyz=0 -0.0612499999999985 0.0610009280869152 rpy=0 0 0, axis 1 0 0, limit lower=-0.17444 upper=0.52358 effort=23.7 velocity=30.0
- added joint R_thigh_joint: type revolute, parent R_hip, child R_thigh, origin xyz=0 -0.01 0 rpy=0 0 0, axis 0 1 0, limit lower=0.0 upper=1.571 effort=23.7 velocity=30.0
- added joint R_wheel_joint: type revolute, parent R_calf, child R_wheel, origin xyz=0 -0.0421817545313912 -0.190000000000001 rpy=0 0 0, axis 0 1 0, limit effort=3.69 velocity=60.0
- added joint depth_cam_joint: type fixed, parent base_link, child depth_cam, origin xyz=0.134942648598871 0 0.120596007530399 rpy=0 0.698131700797732 0, axis 0 0 0

Commit message: Update pineapple version 1 with imu and camera links

File: models/pineapple/pineapple_8dof.urdf (robot description, URDF)
Before this commit: robot pineapple, 10 links, 9 joints
Links:
- removed link depth_cam
- added link cam, mass 0.3; visual mesh filename=package://v1/meshes/cam.STL
- added link imu_link, mass 0.1
- link L_calf: mass 0.50000000 -> 0.5
- link L_hip: mass 0.57300000 -> 0.573
- link L_thigh: mass 0.75000000 -> 0.75
- link L_wheel: mass 0.30500000 -> 0.305
- link R_calf: mass 0.50000000 -> 0.5
- link R_hip: mass 0.57300000 -> 0.573
- link R_thigh: mass 0.75000000 -> 0.75
- link R_wheel: mass 0.30500000 -> 0.305
- link base_link: mass 2.85000000 -> 3.64
Joints:
- removed joint depth_cam_joint
- added joint cam_joint: type fixed, parent base_link, child cam, origin xyz=0.136663127592924 0 0.125539913353642 rpy=0 0.698131700797732 0, axis 0 0 0
- added joint imu_joint: type fixed, parent base_link, child imu_link, origin xyz=0 0 0 rpy=0 0 0, axis 0 0 0
- joint L_calf_joint: origin xyz=0 0.0388671106492234 -0.190000930017623 rpy=0 0 0 -> xyz=0 0.035931787557176 -0.190000001217773 rpy=0 0 0
- joint L_hip_joint: origin xyz=0 0.061249999999998 0.0610009280869146 rpy=0 0 0 -> xyz=0 0.06125 0.065999999287065 rpy=0 0 0
- joint L_thigh_joint: origin xyz=0 0.01 0 rpy=0 0 0 -> xyz=0 0.0129353215081658 0 rpy=0 0 0
- joint L_wheel_joint: origin xyz=0 0.0421817545313912 -0.190000000000001 rpy=0 0 0 -> xyz=0 0.0421817504179199 -0.190000000000001 rpy=0 0 0
- joint R_calf_joint: origin xyz=0 -0.0388671106492234 -0.190000930017624 rpy=0 0 0 -> xyz=0 -0.035931787557176 -0.190000001217773 rpy=0 0 0
- joint R_hip_joint: origin xyz=0 -0.0612499999999985 0.0610009280869152 rpy=0 0 0 -> xyz=0 -0.06125 0.065999999287065 rpy=0 0 0
- joint R_thigh_joint: origin xyz=0 -0.01 0 rpy=0 0 0 -> xyz=0 -0.0129353215081658 0 rpy=0 0 0
- joint R_wheel_joint: origin xyz=0 -0.0421817545313912 -0.190000000000001 rpy=0 0 0 -> xyz=0 -0.0421817504179163 -0.190000000000001 rpy=0 0 0

File: models/pineapple/pineapple_8dof_bp.urdf (robot description, URDF)
Before this commit: robot pineapple, 10 links, 9 joints
Links:
- removed link cam
- added link depth_cam, mass 0.30000000; visual mesh filename=package://v1/meshes/depth_cam.STL
- link base_link: geometry collision mesh filename=package://v1/meshes/base_collision.STL; visual mesh filename=package://v1/meshes/base_link.STL
Joints:
- removed joint cam_joint
- added joint depth_cam_joint: type fixed, parent base_link, child depth_cam, origin xyz=0.134942648598871 0 0.120596007530399 rpy=0 0.698131700797732 0, axis 0 0 0
- joint L_calf_joint: origin xyz=0 0.035931787557176 -0.190000001217773 rpy=0 0 0 -> xyz=0 0.0388671106492234 -0.190000930017623 rpy=0 0 0
- joint L_hip_joint: origin xyz=0 0.06125 0 rpy=0 0 0 -> xyz=0 0.061249999999998 0.0610009280869146 rpy=0 0 0
- joint L_thigh_joint: origin xyz=0 0.0129353215081658 0 rpy=0 0 0 -> xyz=0 0.01 0 rpy=0 0 0
- joint L_wheel_joint: origin xyz=0 0.0421817504179199 -0.190000000000001 rpy=0 0 0 -> xyz=0 0.0421817545313912 -0.190000000000001 rpy=0 0 0
- joint R_calf_joint: origin xyz=0 -0.0359317875571787 -0.190000001217773 rpy=0 0 0 -> xyz=0 -0.0388671106492234 -0.190000930017624 rpy=0 0 0
- joint R_hip_joint: origin xyz=0 -0.0612499999999985 0 rpy=0 0 0 -> xyz=0 -0.0612499999999985 0.0610009280869152 rpy=0 0 0
- joint R_thigh_joint: origin xyz=0 -0.0129353215081659 0 rpy=0 0 0 -> xyz=0 -0.01 0 rpy=0 0 0
- joint R_wheel_joint: origin xyz=0 -0.0421817504179163 -0.190000000000001 rpy=0 0 0 -> xyz=0 -0.0421817545313912 -0.190000000000001 rpy=0 0 0

Commit message: Update pineapple code to new motors

File: models/pineapple/pineapple_8dof.urdf (robot description, URDF)
Before this commit: robot pineapple, 11 links, 10 joints
Links:
- removed link imu_link
- link L_calf: mass 0.5 -> 0.567
- link L_hip: mass 0.573 -> 0.585
- link L_thigh: mass 0.75 -> 0.98
- link L_wheel: mass 0.305 -> 0.3; geometry collision cylinder length=0.023 radius=0.075; visual mesh filename=package://v1/meshes/L_wheel.STL
- link R_calf: mass 0.5 -> 0.567
- link R_hip: mass 0.573 -> 0.585
- link R_thigh: mass 0.75 -> 0.98
- link R_wheel: mass 0.305 -> 0.3; geometry collision cylinder length=0.023 radius=0.075; visual mesh filename=package://v1/meshes/R_wheel.STL
- link base_link: mass 3.64 -> 3.63; geometry collision mesh filename=package://v1/meshes/base_link_collision.STL; visual mesh filename=package://v1/meshes/base_link.STL
Joints:
- removed joint imu_joint
- joint L_calf_joint: limit lower=-3.1416 upper=0.0 effort=33.5 velocity=21.0 -> lower=-3.141 upper=0 effort=23.7 velocity=30.1; origin xyz=0 0.035931787557176 -0.190000001217773 rpy=0 0 0 -> xyz=0 0.04135 -0.165 rpy=0 0 0
- joint L_hip_joint: axis 1 0 0 -> -1 0 0; limit lower=-0.52358 upper=0.17444 effort=23.7 velocity=30.0 -> lower=-0.52358 upper=0.17444 effort=23.7 velocity=30.1; origin xyz=0 0.06125 0.065999999287065 rpy=0 0 0 -> xyz=0 0.061689 0.066 rpy=0 0 0
- joint L_thigh_joint: limit lower=0.0 upper=1.571 effort=23.7 velocity=30.0 -> lower=0 upper=1.57 effort=23.7 velocity=30.1; origin xyz=0 0.0129353215081658 0 rpy=0 0 0 -> xyz=0 0.027596 0 rpy=0 0 0
- joint L_wheel_joint: origin xyz=0 0.0421817504179199 -0.190000000000001 rpy=0 0 0 -> xyz=0 0.024414 -0.165 rpy=0 0 0
- joint R_calf_joint: limit lower=-3.1416 upper=0.0 effort=33.5 velocity=21.0 -> lower=-3.141 upper=0 effort=23.7 velocity=30.1; origin xyz=0 -0.035931787557176 -0.190000001217773 rpy=0 0 0 -> xyz=0 -0.04135 -0.165 rpy=0 0 0
- joint R_hip_joint: axis 1 0 0 -> -1 0 0; limit lower=-0.17444 upper=0.52358 effort=23.7 velocity=30.0 -> lower=-0.17444 upper=0.52358 effort=23.7 velocity=30.1; origin xyz=0 -0.06125 0.065999999287065 rpy=0 0 0 -> xyz=0 -0.061689 0.066 rpy=0 0 0
- joint R_thigh_joint: limit lower=0.0 upper=1.571 effort=23.7 velocity=30.0 -> lower=0 upper=1.57 effort=23.7 velocity=30.1; origin xyz=0 -0.0129353215081658 0 rpy=0 0 0 -> xyz=0 -0.027596 0 rpy=0 0 0
- joint R_wheel_joint: origin xyz=0 -0.0421817504179163 -0.190000000000001 rpy=0 0 0 -> xyz=0 -0.024414 -0.165 rpy=0 0 0
