Commit message: Fix pineapple v3 models

File: models/pineapple/pineapple_v3.urdf (robot description, URDF)
Before this commit: robot v3, 14 links, 13 joints
Links:
- removed link 5dof
- removed link 6dof
- removed link arm_base
- removed link fore_arm
- removed link upper_arm
Joints:
- removed joint 5dof_joint
- removed joint arm_base_joint
- removed joint arm_joint
- removed joint fore_arm_joint
- removed joint upper_arm_joint
