Commit message: WIP not passing all tests, some jacobian issues

File: models/pineapple/pineapple_v3_gripper.urdf (robot description, URDF)
Before this commit: robot v3_gripper, 16 links, 15 joints
Links:
- added link gripper_center, mass 0.001; visual sphere radius=0.005
- link gripper_left_finger: geometry collision box size=0.05 0.016 0.015; visual box size=0.05 0.016 0.015
- link gripper_right_finger: geometry collision box size=0.05 0.016 0.015; visual box size=0.05 0.016 0.015
Joints:
- added joint gripper_center_joint: type fixed, parent 6dof, child gripper_center, origin xyz=0.075 0 -0.04 rpy=1.5708 0 0
- joint gripper_left_joint: origin xyz=0 0.008 -0.073 rpy=0 0 0 -> xyz=-0.025 0.008 0.0 rpy=0 0 0; parent 6dof -> gripper_center
- joint gripper_right_joint: origin xyz=0 -0.008 -0.073 rpy=0 0 0 -> xyz=-0.025 -0.008 0 rpy=0 0 0; parent 6dof -> gripper_center

Commit message: Fix kinematics rotation bugs: custom quat kinematics chain and axis angle taylor expansion

File: models/pineapple/pineapple_v3_gripper.urdf (robot description, URDF)
Before this commit: robot v3_gripper, 17 links, 16 joints
Links:
- link gripper_left_finger: geometry collision box size=0.016 0.016 0.05; visual box size=0.016 0.016 0.05
- link gripper_right_finger: geometry collision box size=0.016 0.016 0.05; visual box size=0.016 0.016 0.05
Joints:
- joint gripper_center_joint: origin xyz=0.075 0 -0.04 rpy=1.5708 0 0 -> xyz=0.075 0 -0.04 rpy=0 0 0
- joint gripper_left_joint: axis 0 1 0 -> 0 0 1; origin xyz=-0.025 0.008 0.0 rpy=0 0 0 -> xyz=-0.025 0 0.008 rpy=0 0 0
- joint gripper_right_joint: axis 0 -1 0 -> 0 0 -1; origin xyz=-0.025 -0.008 0 rpy=0 0 0 -> xyz=-0.025 0 -0.008 rpy=0 0 0

Commit message: Fix gripper orientation

File: models/pineapple/pineapple_v3_gripper.urdf (robot description, URDF)
Before this commit: robot v3_gripper, 17 links, 16 joints
Links:
- link gripper_left_finger: geometry collision box size=0.05 0.016 0.015; visual box size=0.05 0.016 0.015
- link gripper_right_finger: geometry collision box size=0.05 0.016 0.015; visual box size=0.05 0.016 0.015
Joints:
- joint gripper_left_joint: axis 0 0 1 -> 0 1 0; origin xyz=-0.025 0 0.008 rpy=0 0 0 -> xyz=-0.025 0 0.008 rpy=1.5708 0 0
- joint gripper_right_joint: axis 0 0 -1 -> 0 -1 0; origin xyz=-0.025 0 -0.008 rpy=0 0 0 -> xyz=-0.025 0 -0.008 rpy=1.5708 0 0

Commit message: Merge conflicts

File: models/pineapple/pineapple_v3_gripper.urdf (robot description, URDF)
Before this commit: robot v3_gripper, 17 links, 16 joints
Links:
- link 5dof: geometry collision box size=0.065 0.065 0.06; visual mesh filename=package://v3_arm/meshes/5dof.dae scale=1 1 1
- link 6dof: geometry collision box size=0.06 0.065 0.072; visual mesh filename=package://v3_arm/meshes/6dof.dae scale=1 1 1
- link arm_base: geometry visual mesh filename=package://v3_arm/meshes/arm_base.dae scale=1 1 1
- link base_link: geometry collision box size=0.13 0.13 0.04; collision box size=0.23 0.08 0.12
- link calf_l: geometry collision box size=0.07 0.0445 0.295; visual mesh filename=package://v3_arm/meshes/calf_l.dae scale=1 1 1
- link calf_r: geometry collision box size=0.07 0.0445 0.295; visual mesh filename=package://v3_arm/meshes/calf_r.dae scale=1 1 1
- link fore_arm: geometry collision box size=0.26 0.062 0.06; visual mesh filename=package://v3_arm/meshes/fore_arm.dae scale=1 1 1
- link hip_thigh_conn_l: geometry visual mesh filename=package://v3_arm/meshes/hip_thigh_conn.dae scale=1 1 1
- link hip_thigh_conn_r: geometry visual mesh filename=package://v3_arm/meshes/hip_thigh_conn.dae scale=1 1 1
- link thigh_l: geometry collision box size=0.064 0.0675 0.288; visual mesh filename=package://v3_arm/meshes/thigh_l.dae scale=1 1 1
- link thigh_r: geometry collision box size=0.064 0.0675 0.288; visual mesh filename=package://v3_arm/meshes/thigh_r.dae scale=1 1 1
- link upper_arm: geometry collision box size=0.353 0.07 0.068; visual mesh filename=package://v3_arm/meshes/upper_arm.dae scale=1 1 1
- link wheel_l: geometry collision cylinder length=0.035 radius=0.0925; visual mesh filename=package://v3_arm/meshes/wheel_l.dae scale=1 1 1
- link wheel_r: geometry collision cylinder length=0.035 radius=0.0925; visual mesh filename=package://v3_arm/meshes/wheel_r.dae scale=1 1 1
